File: kicad/testkicad.kicad_pcb (KiCad board)
At the start: 2 copper layers, 11 parts, among them SW1 SW_PUSH

Commit message: ...
Parts:
- CONN1: value FT232_CONN -> FT232; footprint Pin_Headers:Pin_Header_Angled_1x06 -> Pin_Headers:Pin_Header_Straight_1x06
- CONN2: footprint Pin_Headers:Pin_Header_Angled_1x11 -> Pin_Headers:Pin_Header_Straight_1x11
- R1, R2, R3, R4, R5: footprint Resistors_ThroughHole:Resistor_Horizontal_RM7mm -> Resistors_ThroughHole:Resistor_Vertical_RM5mm
- SW1: value SW_PUSH -> RESET
- moved R2 39.2 mm to (149.4, 43.7), turned to 0 degrees
- moved R5 31.7 mm to (176.8, 28.4), turned to 0 degrees
- moved R4 30.1 mm to (169.7, 58.9), turned to 90 degrees
- moved R1 28.1 mm to (162.1, 58.9), turned to 90 degrees
- moved CONN1 27.5 mm to (135.1, 39.1)
- moved C1 26.2 mm to (148.8, 35.6), turned to 270 degrees
- moved R3 25.4 mm to (165.6, 58.9), turned to 90 degrees
- moved SW1 22.8 mm to (148.8, 31.5), turned to 180 degrees
- moved ESP1 22.0 mm to (158.5, 38.1), turned to 0 degrees
- moved ADC1 8.65 mm to (186.9, 51.3)
- moved CONN2 8.65 mm to (203.2, 51.3)
Connections:
- net Net-(ADC1-Pad10) renamed /GPIO15
- net Net-(ADC1-Pad11) renamed /MOSI
- net Net-(ADC1-Pad12) renamed /MISO
- net Net-(ADC1-Pad13) renamed /SPI_CLK
- net Net-(ADC1-Pad15) renamed +3V3
- net Net-(CONN1-Pad4) renamed /ESP_RX
- net Net-(CONN1-Pad5) renamed /ESP_TX
- net Net-(ESP1-Pad11) renamed /GPIO2
- net Net-(ESP1-Pad12) renamed /GPIO0
- C1 pad 1: Net-(C1-Pad1) -> /REST
- ESP1 pad 1: Net-(C1-Pad1) -> /REST
- ESP1 pad 3: Net-(ESP1-Pad3) -> /CH_PD
- ESP1 pad 4: Net-(C1-Pad1) -> /GPIO16
- R1 pad 2: Net-(C1-Pad1) -> /CH_PD
- R2 pad 2: Net-(ESP1-Pad3) -> /REST
- SW1 pad 1: GND -> /REST
- SW1 pad 2: Net-(C1-Pad1) -> GND
Routing:
- net /ESP_RX: track 0.00 -> 146.7 mm
- net +3V3: track 4.48 -> 77.0 mm
- net /ESP_TX: track 0.00 -> 43.7 mm
- net /GPIO15: track 0.00 -> 33.7 mm
- net /REST: track 0.00 -> 25.2 mm
- net /CH_PD: track 0.00 -> 16.6 mm
- net Net-(ADC1-Pad8): track 0.00 -> 16.3 mm
- net Net-(ADC1-Pad7): track 0.00 -> 16.3 mm
- net Net-(ADC1-Pad6): track 0.00 -> 16.3 mm
- net Net-(ADC1-Pad5): track 0.00 -> 16.3 mm
- net Net-(ADC1-Pad4): track 0.00 -> 16.3 mm
- net Net-(ADC1-Pad3): track 0.00 -> 16.3 mm
- net Net-(ADC1-Pad2): track 0.00 -> 16.3 mm
- net Net-(ADC1-Pad1): track 0.00 -> 16.3 mm
- net /GPIO0: track 0.00 -> 14.4 mm
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- added copper zone on F.Cu, net GND

Commit message: ...
Parts:
- moved R4 33.6 mm to (161.0, 26.4), turned to 180 degrees
- moved R3 32.8 mm to (170.2, 26.4), turned to 180 degrees
- moved R1 19.3 mm to (181.4, 58.9), turned to 180 degrees
- moved ESP1 16.8 mm to (173.2, 46.2), turned to 180 degrees
- moved C1 13.1 mm to (151.9, 48.3)
- moved ADC1 7.62 mm to (194.6, 51.3)
- moved R2 5.00 mm to (144.8, 45.7)
- moved R5 3.70 mm to (180.3, 27.4)
- moved SW1 0.51 mm to (148.8, 31.0)
Routing:
- net /ESP_RX: track 146.7 -> 0.00 mm
- net +3V3: track 77.0 -> 0.00 mm
- net /ESP_TX: track 43.7 -> 0.00 mm
- net /GPIO15: track 33.7 -> 0.00 mm
- net /REST: track 25.2 -> 0.00 mm
- net /CH_PD: track 16.6 -> 0.00 mm
- net Net-(ADC1-Pad8): track 16.3 -> 0.00 mm
- net Net-(ADC1-Pad7): track 16.3 -> 0.00 mm
- net Net-(ADC1-Pad6): track 16.3 -> 0.00 mm
- net Net-(ADC1-Pad5): track 16.3 -> 0.00 mm
- net Net-(ADC1-Pad4): track 16.3 -> 0.00 mm
- net Net-(ADC1-Pad3): track 16.3 -> 0.00 mm
- net Net-(ADC1-Pad2): track 16.3 -> 0.00 mm
- net Net-(ADC1-Pad1): track 16.3 -> 0.00 mm
- net /GPIO0: track 14.4 -> 0.00 mm
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